File: hardware/nrfmicro.kicad_pcb (KiCad board)
At the start: 2 copper layers, 18.1 x 33.3 mm, 24 parts, among them J1 USB-C Conn, J2 SWD, J3 Ex_Bat, J4 Ex_USB, Q1 AO3407, Q2 AO3407, U1 E73-2G4M08S1C, U2 XC6220B331MR-G, U3 TP4054, U4 ProMicro, X1 32.768kHz

Commit message: starting to modify, lots to do still
Parts:
- removed G***: LOGO, Custom Parts:Catmelon_Small
- removed J1: USB-C Conn, nrfmicro:USB-C_C168688
- removed U4: ProMicro, nrfmicro:pro_micro
- added U5: ATmega32A-P, Package_DIP:DIP-40_W15.24mm, F.Cu at (57.1, 45.1)
- J2, J4: moved to B.Cu
- moved J3 79.9 mm to (105.4, 38.7), turned to 90 degrees
- moved J2 68.6 mm to (95.2, 35.7), turned to 270 degrees
- moved J4 65.4 mm to (95.2, 40.5), turned to 270 degrees
- moved D1 52.6 mm to (79.8, 35.1)
- moved Q1 52.6 mm to (74.7, 35.0)
- moved R1 52.6 mm to (77.0, 35.0)
- moved R3 52.6 mm to (81.3, 35.0)
- moved R4 52.6 mm to (75.4, 38.2)
- moved R7 52.6 mm to (78.2, 40.6)
- moved R9 52.6 mm to (82.6, 35.0)
- moved U3 52.6 mm to (81.7, 38.2)
- moved D3 52.6 mm to (85.8, 38.2)
- moved Q2 52.6 mm to (84.8, 35.0)
- moved R2 52.6 mm to (78.3, 35.0)
- moved R5 52.6 mm to (81.3, 40.6)
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Routing:
- net GND: track 116.4 -> 17.1 mm, vias 2 -> 0
- net DATA+: track 39.2 -> 0.05 mm, vias 2 -> 1
- net DATA-: track 37.0 -> 1.22 mm
- net BLUE_LED: track 26.4 -> 0.67 mm
- net nRF_VDD: track 32.4 -> 6.64 mm
- net VBUS: track 49.5 -> 24.3 mm, vias 5 -> 4
- net RESET: track 22.5 -> 0.00 mm, vias 3 -> 0
- net /P0.06: track 22.2 -> 0.00 mm
- net /P0.08: track 18.7 -> 0.00 mm
- net POWER_PIN: track 22.0 -> 11.6 mm
- net SWC: track 9.81 -> 0.00 mm, vias 1 -> 0
- net BATTERY_PIN: track 9.56 -> 1.26 mm
- net /P0.15: track 8.13 -> 0.00 mm
- net VBAT: track 34.8 -> 27.0 mm
- net /P0.17: track 6.82 -> 0.00 mm
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