File: hardware/NumDisciplineBLE.kicad_pcb (KiCad board)
At the start: 2 copper layers, 18.1 x 33.3 mm, 22 parts, among them J2 SWD, J3 Ex_Bat, J4 Ex_USB, Q1 AO3407, Q2 AO3407, U1 E73-2G4M08S1C, U2 XC6220B331MR-G, U3 TP4054, U5 ATmega32A-P, X1 32.768kHz

Commit message: basic layout done
Parts:
- removed U5: ATmega32A-P, Package_DIP:DIP-40_W15.24mm
- added J1: Conn_02x20_Counter_Clockwise, nrfmicro:2x20_P2.54mm_Vertical_SMD_reversed, B.Cu at (119.4, 38.7)
- moved U1 74.4 mm to (126.3, 37.2)
- moved Q1 48.6 mm to (123.2, 31.1), turned to 90 degrees
- moved R1 46.2 mm to (123.2, 33.7), turned to 180 degrees
- moved D2 46.1 mm to (119.4, 31.5), turned to 0 degrees
- moved R2 44.9 mm to (123.2, 35.3), turned to 180 degrees
- moved R4 44.3 mm to (119.4, 33.0), turned to 0 degrees
- moved D1 43.4 mm to (123.2, 37.1), turned to 180 degrees
- moved R3 42.1 mm to (123.2, 38.9), turned to 180 degrees
- moved U2 41.7 mm to (119.5, 35.6), turned to 180 degrees
- moved R6 41.3 mm to (116.3, 34.5), turned to 270 degrees
- moved R9 40.9 mm to (123.2, 40.4), turned to 180 degrees
- moved Q2 39.2 mm to (123.2, 42.9), turned to 270 degrees
- moved R7 38.2 mm to (116.3, 37.4), turned to 270 degrees
- moved U3 37.8 mm to (119.5, 39.4), turned to 180 degrees
- moved R8 35.5 mm to (119.5, 42.2), turned to 0 degrees
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Routing:
- net DATA+: track 0.05 -> 0.00 mm, vias 1 -> 0
- net VBUS: track 24.3 -> 24.4 mm, vias 4 -> 5
Other:
- board outline removed
- board text removed: "nRFMicro 1.4"

Commit message: pre-routing
Parts:
- moved R5 5.08 mm to (111.2, 40.5)
- moved R6 5.08 mm to (111.2, 34.5)
- moved R7 5.08 mm to (111.2, 37.4)
- moved X1 5.08 mm to (111.4, 43.8)
- moved D3 2.54 mm to (116.9, 43.7)
- moved R8 2.54 mm to (116.9, 42.2)
- moved U2 2.54 mm to (117.0, 35.6)
- moved U3 2.54 mm to (117.0, 39.4)
- moved D2 2.54 mm to (116.8, 31.5)
- moved R4 2.54 mm to (116.8, 33.0)
Routing:
- net VBAT: track 27.0 -> 0.00 mm, vias 3 -> 0
- net VBUS: track 24.4 -> 0.00 mm, vias 5 -> 0
- net GND: track 17.1 -> 0.00 mm
- net Net-(D1-Pad1): track 13.1 -> 0.00 mm, vias 2 -> 0
- net POWER_PIN: track 11.6 -> 0.00 mm, vias 2 -> 0
- net nRF_VDD: track 6.64 -> 0.00 mm, vias 2 -> 0
- net Net-(D2-Pad1): track 2.09 -> 0.00 mm
- net Net-(R8-Pad2): track 1.73 -> 0.00 mm
- net Net-(D3-Pad1): track 1.58 -> 0.00 mm
- net Net-(R5-Pad1): track 1.56 -> 0.00 mm
- net BATTERY_PIN: track 1.26 -> 0.00 mm
- net DATA-: track 1.22 -> 0.00 mm, vias 2 -> 0
- net BLUE_LED: track 0.67 -> 0.00 mm
- added copper zone on B.Cu, net GND
- added copper zone on F.Cu, net GND

Commit message: pre-routing2
Parts:
- removed R2, R3: 5.1K, Resistor_SMD:R_0603_1608Metric
- moved J2 26.7 mm to (124.5, 35.1), turned to 180 degrees
- moved Q1 25.8 mm to (97.8, 35.8), turned to 180 degrees
- moved J4 25.4 mm to (122.4, 35.1), turned to 180 degrees
- moved D1 23.6 mm to (99.7, 38.7)
- moved X1 17.8 mm to (126.7, 34.8), turned to 90 degrees
- moved D3 17.3 mm to (99.8, 40.9), turned to 180 degrees
- moved U2 15.4 mm to (101.6, 35.8), turned to 0 degrees
- moved R8 14.0 mm to (103.0, 40.9)
- moved R1 12.0 mm to (112.5, 39.1), turned to 270 degrees
- moved U3 11.6 mm to (105.9, 35.8)
- moved R4 9.96 mm to (109.0, 39.1), turned to 90 degrees
- moved D2 9.74 mm to (110.7, 39.1), turned to 90 degrees
- moved R5 7.54 mm to (103.9, 38.9), turned to 180 degrees
- moved R9 7.00 mm to (117.3, 36.6), turned to 0 degrees
- moved Q2 6.97 mm to (117.3, 39.1), turned to 0 degrees
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Routing:
- removed copper zone on F.Cu, net GND

Commit message: post-autoroute
Routing:
- net /P0.22: track 0.00 -> 71.7 mm
- net VBUS: track 0.00 -> 69.3 mm
- net /P1.00: track 0.00 -> 59.8 mm
- net /P1.06: track 0.00 -> 57.6 mm, vias 0 -> 1
- net /P0.10: track 0.00 -> 54.0 mm, vias 0 -> 1
- net /P1.02: track 0.00 -> 50.9 mm
- net nRF_VDD: track 0.00 -> 50.5 mm, vias 0 -> 1
- net /P0.09: track 0.00 -> 47.1 mm, vias 0 -> 1
- net /P1.04: track 0.00 -> 44.3 mm, vias 0 -> 1
- net /P0.08: track 0.00 -> 43.6 mm
- net /P0.13: track 0.00 -> 41.0 mm, vias 0 -> 1
- net /P0.06: track 0.00 -> 40.1 mm
- net /P0.24: track 0.00 -> 38.8 mm, vias 0 -> 1
- net BLUE_LED: track 0.00 -> 34.7 mm
- net /P0.17: track 0.00 -> 32.9 mm, vias 0 -> 1
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
Commit message: first gerbers
Routing:
- net GND: track 16.5 -> 99.5 mm, vias 6 -> 18
- net DATA+: track 17.1 -> 23.4 mm
- net DATA-: track 20.0 -> 23.5 mm
- net /P0.03: track 16.5 -> 18.3 mm
- net /P0.13: track 41.0 -> 42.8 mm
- net nRF_VDD: track 50.5 -> 51.8 mm
- net /P0.24: track 38.8 -> 38.1 mm
- net /P0.08: track 43.6 -> 42.9 mm
- net /P0.07: track 15.2 -> 14.7 mm
Other:
- board outline added: 53.3 x 24.1 mm
- net class Power: clearance 0.2 -> 0.3

Commit message: R0 done
Routing:
- net GND: track 99.5 -> 100.1 mm
Other:
- board text added: "NumDiscipline BLE ERL 06Nov2020 R0"
Changed lines of the file:
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@@
   (general
     (thickness 1.6)
-    (drawings 8)
+    (drawings 9)
     (tracks 487)
     (zones 0)
@@
     )
   )
+  (gr_text "NumDiscipline BLE\nERL 06Nov2020 R0" (at 93.599 48.641) (layer F.SilkS)
+    (effects (font (size 0.7 0.7) (thickness 0.08)) (justify left))
+  )
   (gr_line (start 146.05 27.305) (end 146.05 50.165) (layer Edge.Cuts) (width 0.15))
   (gr_arc (start 93.345 27.305) (end 93.345 26.67) (angle -90) (layer Edge.Cuts) (width 0.15))
@@
   (segment (start 130.914 42.395) (end 130.108 42.395) (width 0.2) (layer F.Cu) (net 1) (status 20))
   (segment (start 130.937 42.418) (end 130.914 42.395) (width 0.2) (layer F.Cu) (net 1))
-  (via (at 113.792 32.385) (size 0.6) (drill 0.33) (layers F.Cu B.Cu) (net 1))
-  (via (at 114.681 29.845) (size 0.6) (drill 0.33) (layers F.Cu B.Cu) (net 1))
-  (segment (start 113.792 30.734) (end 114.681 29.845) (width 0.2) (layer F.Cu) (net 1))
-  (segment (start 113.792 32.385) (end 113.792 30.734) (width 0.2) (layer F.Cu) (net 1))
-  (via (at 131.191 28.702) (size 0.6) (drill 0.33) (layers F.Cu B.Cu) (net 1))
-  (segment (start 116.123999 28.402001) (end 114.681 29.845) (width 0.2) (layer F.Cu) (net 1))
-  (segment (start 130.891001 28.402001) (end 116.123999 28.402001) (width 0.2) (layer F.Cu) (net 1))
-  (segment (start 131.191 28.702) (end 130.891001 28.402001) (width 0.2) (layer F.Cu) (net 1))
   (segment (start 117.233063 38.866001) (end 118.11 37.989064) (width 0.2) (layer F.Cu) (net 1))
   (segment (start 114.525699 38.866001) (end 117.233063 38.866001) (width 0.2) (layer F.Cu) (net 1))
@@
   (segment (start 99.695 29.21) (end 99.695 29.083) (width 0.2) (layer F.Cu) (net 1))
   (segment (start 101.219 30.734) (end 99.695 29.21) (width 0.2) (layer F.Cu) (net 1))
+  (segment (start 118.11 29.465) (end 117.095 29.465) (width 0.2) (layer B.Cu) (net 1) (status 10))
+  (segment (start 117.095 29.465) (end 116.713 29.083) (width 0.2) (layer B.Cu) (net 1))
+  (segment (start 113.792 32.004) (end 113.792 32.385) (width 0.2) (layer F.Cu) (net 1))
+  (segment (start 116.713 29.083) (end 113.792 32.004) (width 0.2) (layer F.Cu) (net 1))
+  (via (at 116.713 29.083) (size 0.6) (drill 0.33) (layers F.Cu B.Cu) (net 1))
+  (via (at 131.191 28.702) (size 0.6) (drill 0.33) (layers F.Cu B.Cu) (net 1))
+  (via (at 113.792 32.385) (size 0.6) (drill 0.33) (layers F.Cu B.Cu) (net 1))
+  (segment (start 130.81 29.083) (end 116.713 29.083) (width 0.2) (layer F.Cu) (net 1))
+  (segment (start 131.191 28.702) (end 130.81 29.083) (width 0.2) (layer F.Cu) (net 1))
   (via (at 120.015 44.577) (size 0.6) (drill 0.33) (layers F.Cu B.Cu) (net 2))
   (segment (start 130.616 44.727) (end 130.3691 44.4801) (width 0.2) (layer F.Cu) (net 2) (status 30))
@@
   (segment (start 121.0834 44.4801) (end 120.9865 44.577) (width 0.2) (layer F.Cu) (net 2))
   (segment (start 120.015 44.577) (end 120.015 45.6565) (width 0.2) (layer B.Cu) (net 2))
-  (segment (start 117.5395 48.132) (end 115.697 48.132) (width 0.2) (layer B.Cu) (net 2))
+  (segment (start 117.5395 48.132) (end 115.697 48.132) (width 0.2) (layer B.Cu) (net 2) (status 20))
   (segment (start 120.015 45.6565) (end 117.5395 48.132) (width 0.2) (layer B.Cu) (net 2))
   (segment (start 134.426 31.6887) (end 129.9717 31.6887) (width 0.2) (layer F.Cu) (net 3))
@@
   (segment (start 133.709764 48.132) (end 136.017 48.132) (width 0.2) (layer B.Cu) (net 12) (status 20))
   (segment (start 131.805764 46.228) (end 133.709764 48.132) (width 0.2) (layer B.Cu) (net 12))
-  (segment (start 131.3815 46.228) (end 131.805764 46.228) (width 0.2) (layer B.Cu) (net 12))
+  (segment (start 127.762 46.228) (end 131.805764 46.228) (width 0.2) (layer B.Cu) (net 12))
   (segment (start 127.762 46.228) (end 127.381 45.847) (width 0.2) (layer B.Cu) (net 12))
   (segment (start 127.381 45.847) (end 127.508 45.974) (width 0.2) (layer B.Cu) (net 12))
-  (segment (start 131.3815 46.228) (end 127.762 46.228) (width 0.2) (layer B.Cu) (net 12))
   (segment (start 127.127 45.552002) (end 127.381 45.847) (width 0.2) (layer B.Cu) (net 12))
   (via (at 131.3815 46.1645) (size 0.6) (layers F.Cu B.Cu) (net 12))
@@
   (segment (start 115.731999 29.244999) (end 117.221 30.734) (width 0.2) (layer B.Cu) (net 15))
   (segment (start 113.73 29.465) (end 113.950001 29.244999) (width 0.2) (layer B.Cu) (net 15))
-  (segment (start 113.03 29.465) (end 113.73 29.465) (width 0.2) (layer B.Cu) (net 15))
+  (segment (start 113.03 29.465) (end 113.73 29.465) (width 0.2) (layer B.Cu) (net 15) (status 10))
   (segment (start 117.221 30.734) (end 121.774101 30.715101) (width 0.2) (layer B.Cu) (net 15))
   (segment (start 135.696 44.727) (end 135.696 45.475402) (width 0.2) (layer F.Cu) (net 16) (status 10))
@@
   (segment (start 111.487001 30.715001) (end 110.237 29.465) (width 0.2) (layer B.Cu) (net 20))
   (segment (start 116.186001 30.715001) (end 111.487001 30.715001) (width 0.2) (layer B.Cu) (net 20))
-  (segment (start 110.237 29.465) (end 107.95 29.465) (width 0.2) (layer B.Cu) (net 20))
+  (segment (start 110.237 29.465) (end 107.95 29.465) (width 0.2) (layer B.Cu) (net 20) (status 20))
   (segment (start 116.58631 31.11531) (end 116.186001 30.715001) (width 0.2) (layer B.Cu) (net 20))
   (segment (start 117.8573 32.0636) (end 116.90901 31.11531) (width 0.2) (layer B.Cu) (net 20))
@@
   (segment (start 139.101 43.4493) (end 138.998 43.4493) (width 0.2) (layer B.Cu) (net 36))
   (segment (start 141.07882 50.02498) (end 141.8974 49.2064) (width 0.2) (layer B.Cu) (net 36))
-  (segment (start 138.998 43.4493) (end 138.998 42.649) (width 0.2) (layer B.Cu) (net 36))
+  (segment (start 138.998 43.4493) (end 138.998 42.649) (width 0.2) (layer B.Cu) (net 36) (status 20))
   (segment (start 141.8974 49.2064) (end 141.8974 46.2457) (width 0.2) (layer B.Cu) (net 36))
   (segment (start 100.5633 49.3823) (end 101.20598 50.02498) (width 0.2) (layer B.Cu) (net 36))
   (segment (start 100.457 49.3823) (end 100.5633 49.3823) (width 0.2) (layer B.Cu) (net 36))
-  (segment (start 100.457 48.132) (end 100.457 49.3823) (width 0.2) (layer B.Cu) (net 36))
+  (segment (start 100.457 48.132) (end 100.457 49.3823) (width 0.2) (layer B.Cu) (net 36) (status 10))
   (segment (start 138.557 44.832) (end 138.557 43.5817) (width 0.2) (layer B.Cu) (net 37) (status 10))
   (segment (start 130.108 39.855) (end 132.394 39.855) (width 0.2) (layer B.Cu) (net 37) (status 10))
@@
   (segment (start 134.2774 43.852402) (end 134.2774 43.5609) (width 0.2) (layer B.Cu) (net 39))
   (segment (start 138.556998 48.132) (end 134.2774 43.852402) (width 0.2) (layer B.Cu) (net 39))
-  (segment (start 141.097 48.132) (end 138.556998 48.132) (width 0.2) (layer B.Cu) (net 39))
+  (segment (start 141.097 48.132) (end 138.556998 48.132) (width 0.2) (layer B.Cu) (net 39) (status 10))
   (segment (start 125.4501 38.7045) (end 127.0332 38.7045) (width 0.3) (layer F.Cu) (net 40))
   (segment (start 127.0332 38.7045) (end 127.5467 39.218) (width 0.3) (layer F.Cu) (net 40))
